File: PCB/PWM_amp/PWM_amp.kicad_pcb (KiCad board)
At the start: 2 copper layers, 84 x 84 mm, 47 parts, among them J1 Conn_01x06_Pin, J10 XT30UPB-M, J2 Conn_01x06_Pin, J3 Conn_01x02_Pin, J4 Conn_01x02_Pin, J49 XT60PW-M, J5 XT30UPB-M, Q1 FDD8447L, Q2 FDD8447L, U1 VNH5019A-E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

Commit message: 3d models and PCB
Parts:
- removed CS (x2): CS, TestPoint:TestPoint_Loop_D1.80mm_Drill1.0mm_Beaded
- added C4: 1uF, Capacitor_SMD:C_0805_2012Metric_Pad1.18x1.45mm_HandSolder, F.Cu at (226.8, 116.4)
- added C6: 1uF, Capacitor_SMD:C_0805_2012Metric_Pad1.18x1.45mm_HandSolder, F.Cu at (233.9, 88.1)
- added C7: 0.1uF, Capacitor_SMD:C_0805_2012Metric_Pad1.18x1.45mm_HandSolder, F.Cu at (231.5, 146.7)
- added C8: 0.1uF, Capacitor_SMD:C_0805_2012Metric_Pad1.18x1.45mm_HandSolder, F.Cu at (231.6, 114.7)
- added G***: LOGO, LOGO, F.Cu at (266.9, 104.3)
- added G***: LOGO, LOGO, F.Cu at (235.9, 96.8)
- added G***: LOGO, LOGO, F.Cu at (267.7, 85.7)
- added G***: LOGO, LOGO, B.Cu at (267.7, 85.7)
- moved H1 65.7 mm to (263.6, 153.9), turned to -90 degrees
- moved H2 63.4 mm to (200.6, 153.9), turned to -90 degrees
- moved H8 62.7 mm to (263.6, 90.9), turned to -90 degrees
- moved OUT1 61.1 mm to (196.1, 95.4), turned to -90 degrees
- moved H3 60.3 mm to (200.6, 90.9), turned to -90 degrees
- moved OUT1 54.7 mm to (193.2, 129.6), turned to -90 degrees
- moved C3 51.3 mm to (212.0, 90.1), turned to 180 degrees
- moved J49 51.2 mm to (263.7, 105.6), turned to 90 degrees
- moved PGND 51.1 mm to (245.9, 88.0), turned to -90 degrees
- moved OUT2 49.9 mm to (222.2, 155.1), turned to -90 degrees
- moved J5 49.5 mm to (196.1, 117.8), turned to 180 degrees
- moved J3 48.9 mm to (203.5, 99.9), turned to 180 degrees
- moved VM 48.0 mm to (239.3, 88.0), turned to -90 degrees
- moved INB1 47.8 mm to (246.9, 148.7), turned to -90 degrees
- moved J10 47.5 mm to (215.0, 150.5), turned to 180 degrees
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Connections:
- J2 pad 1: Net-(J2-Pin_1) -> INB2
- J2 pad 4: +3V_1 -> Net-(J2-Pin_4)
- J2 pad 5: GND1 -> +3V_1
- J2 pad 6: INB2 -> GND1
- R1 pad 1: Net-(J2-Pin_1) -> Net-(J2-Pin_2)
- R12 pad 1: +3V_1 -> Net-(J2-Pin_4)
- R12 pad 2: Net-(U1-CS_DIS) -> Net-(U1-CS)
- R4 pad 1: +3V_1 -> Net-(J1-Pin_4)
- R4 pad 2: Net-(U2-CS_DIS) -> Net-(U2-CS)
- R7 pad 1: Net-(J1-Pin_3) -> GND1
- R7 pad 2: Net-(U2-CS_DIS) -> Net-(U2-CS)
- R8 pad 1: Net-(J2-Pin_1) -> Net-(J2-Pin_2)
- R9 pad 1: Net-(J2-Pin_2) -> GND1
- R9 pad 2: Net-(U1-CS_DIS) -> Net-(U1-CS)
- U1 pad 6: Net-(U1-CS_DIS) -> Net-(J2-Pin_3)
- U1 pad 8: Net-(J2-Pin_3) -> Net-(U1-CS)
- U2 pad 6: Net-(U2-CS_DIS) -> Net-(J1-Pin_3)
- U2 pad 8: Net-(J1-Pin_4) -> Net-(U2-CS)
Routing:
- net Net-(Q1-D): track 12.2 -> 32.5 mm, vias 43 -> 34
- net Net-(J1-Pin_4): track 24.6 -> 5.72 mm
- net Net-(J2-Pin_1): track 18.2 -> 0.00 mm
- net +3V_1: track 91.4 -> 75.3 mm, vias 6 -> 4
- net Net-(Q2-D): track 12.2 -> 28.1 mm, vias 38 -> 34
- net Net-(J2-Pin_2): track 4.04 -> 19.9 mm
- net Net-(U1-CS_DIS): track 11.5 -> 0.00 mm
- net Net-(U2-CS): track 0.00 -> 11.3 mm
- net Net-(U1-CS): track 0.00 -> 11.0 mm
- net Net-(J1-Pin_3): track 6.35 -> 16.7 mm
- net Net-(U2-CS_DIS): track 9.43 -> 0.00 mm
- net Net-(J2-Pin_3): track 26.1 -> 18.1 mm
- net VM1: track 63.0 -> 57.2 mm, vias 0 -> 67
- net Net-(J2-Pin_4): track 0.00 -> 5.74 mm
- net INB2: track 36.8 -> 40.2 mm
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- added copper zone on In1.Cu, net GND1
- added copper zone on B.Cu, net Net-(J3-Pin_2)
- added copper zone on B.Cu, net Net-(J4-Pin_2)
- added copper zone on In2.Cu, net Net-(Q1-D)
- added copper zone on In2.Cu, net Net-(Q2-D)
- added copper zone on In1.Cu, net PGND1
- added copper zone on In2.Cu, net VM1
- removed copper zone on B.Cu, net GND1
Other:
- outline, holes or cut-outs redrawn
- copper layers 2 -> 4
- board text added: "!"
- board text added: "24V"
- board text added: "4/Mar 2026 Iter. 1.1.0"
- board text added: "<<< 15A"
- board text added: "EN > pulled high (enabled) CS_DIS > floating (CS enabled)"
- board text added: "J3"
- board text added: "M3"
- board text removed: "1/Mar 2026 Ver. 1.0"
- board text removed: "EN > pulled high (enabled) CS_DIS > pulled high (CS disabled)"

Commit message: V2 started
Parts:
- removed Q1, Q2: FDD8447L, Package_TO_SOT_SMD:TO-252-2
- added C10: 0.1uF, Capacitor_SMD:C_0805_2012Metric_Pad1.18x1.45mm_HandSolder, F.Cu at (234.5, 101.5)
- added C9: 0.1uF, Capacitor_SMD:C_0805_2012Metric_Pad1.18x1.45mm_HandSolder, F.Cu at (234.5, 132.5)
- moved C4 5.76 mm to (229.8, 121.3), turned to 90 degrees
- moved C6 4.60 mm to (229.7, 89.9), turned to 90 degrees
- moved C3 3.51 mm to (215.5, 90.1)
- moved C5 3.51 mm to (215.4, 121.1)
Routing:
- net VM1: track 57.2 -> 12.0 mm, vias 67 -> 63
- net Net-(U2-CP): track 13.6 -> 3.90 mm
- net Net-(U1-CP): track 13.5 -> 3.97 mm
- net (no net): track 123.3 -> 128.9 mm
- net PGND1: track 3.09 -> 8.27 mm, vias 211 -> 208
- net Net-(C5-Pad1): track 32.5 -> 29.6 mm, vias 34 -> 18
- net Net-(C3-Pad1): track 28.1 -> 25.5 mm, vias 34 -> 20

Commit message: code testing for V2
Parts:
- removed C10, C9: 0.1uF, Capacitor_SMD:C_0805_2012Metric_Pad1.18x1.45mm_HandSolder
- added Q1: FDD8447L, Package_TO_SOT_SMD:TO-252-2, F.Cu at (224.5, 120.9)
- added Q2: FDD8447L, Package_TO_SOT_SMD:TO-252-2, F.Cu at (224.6, 89.9)
- moved C4 5.76 mm to (226.8, 116.4), turned to 180 degrees
- moved C6 4.60 mm to (233.9, 88.1), turned to 45 degrees
- moved C3 3.51 mm to (212.0, 90.1)
- moved C5 3.51 mm to (211.9, 121.1)
Routing:
- net VM1: track 12.0 -> 57.2 mm, vias 63 -> 67
- net Net-(Q1-G): track 3.90 -> 13.6 mm
- net Net-(Q2-G): track 3.97 -> 13.5 mm
- net (no net): track 128.9 -> 123.3 mm
- net PGND1: track 8.27 -> 3.09 mm, vias 208 -> 211
- net Net-(Q1-D): track 29.6 -> 32.5 mm, vias 18 -> 34
- net Net-(Q2-D): track 25.5 -> 28.1 mm, vias 20 -> 34

Commit message: DONE DRAFT
Parts:
- removed INA1: INB1, TestPoint:TestPoint_Loop_D1.80mm_Drill1.0mm_Beaded
- removed INA2: INB2, TestPoint:TestPoint_Loop_D1.80mm_Drill1.0mm_Beaded
- removed INB1: INA1, TestPoint:TestPoint_Loop_D1.80mm_Drill1.0mm_Beaded
- removed INB2: INA2, TestPoint:TestPoint_Loop_D1.80mm_Drill1.0mm_Beaded
- removed J2: Conn_01x06_Pin, Connector_PinHeader_2.54mm:PinHeader_1x06_P2.54mm_Vertical
- removed OUT1 (x2): OUTB, TestPoint:TestPoint_Loop_D1.80mm_Drill1.0mm_Beaded
- removed OUT2 (x2): OUTA, TestPoint:TestPoint_Loop_D1.80mm_Drill1.0mm_Beaded
- removed PGND: GND1, TestPoint:TestPoint_Loop_D1.80mm_Drill1.0mm_Beaded
- removed VM: VM1, TestPoint:TestPoint_Loop_D1.80mm_Drill1.0mm_Beaded
- added J6: Conn_01x07_Pin, Connector_PinSocket_2.54mm:PinSocket_1x07_P2.54mm_Vertical, F.Cu at (243.3, 151.2)
- added R13: 4.7k, Resistor_SMD:R_0805_2012Metric_Pad1.20x1.40mm_HandSolder, B.Cu at (233.1, 138.0)
- added R14: 1k, Resistor_SMD:R_0805_2012Metric_Pad1.20x1.40mm_HandSolder, B.Cu at (235.9, 136.9)
- added R15: 1k, Resistor_SMD:R_0805_2012Metric_Pad1.20x1.40mm_HandSolder, B.Cu at (235.6, 105.9)
- added R16: 4.7k, Resistor_SMD:R_0805_2012Metric_Pad1.20x1.40mm_HandSolder, B.Cu at (232.8, 107.0)
- added TP1: TestPoint, TestPoint:TestPoint_Pad_D1.5mm, F.Cu at (240.3, 150.8)
- added TP10: TestPoint, TestPoint:TestPoint_Plated_Hole_D2.0mm, F.Cu at (294.7, 100.4)
- added TP11: TestPoint, TestPoint:TestPoint_Plated_Hole_D2.0mm, F.Cu at (294.7, 105.5)
- added TP12: TestPoint, TestPoint:TestPoint_Plated_Hole_D2.0mm, F.Cu at (239.3, 88.1)
- added TP2: TestPoint, TestPoint:TestPoint_Pad_D1.5mm, F.Cu at (238.1, 151.9)
- added TP3: TestPoint, TestPoint:TestPoint_Plated_Hole_D2.0mm, F.Cu at (245.9, 88.1)
- added TP4: TestPoint, TestPoint:TestPoint_Pad_D1.5mm, F.Cu at (240.3, 104.8)
- added TP5: TestPoint, TestPoint:TestPoint_Pad_D1.5mm, F.Cu at (246.4, 118.8)
- added TP6: TestPoint, TestPoint:TestPoint_Pad_D1.5mm, F.Cu at (240.3, 135.4)
- added TP7: TestPoint, TestPoint:TestPoint_Pad_D1.5mm, F.Cu at (240.3, 120.8)
- added TP8: TestPoint, TestPoint:TestPoint_Plated_Hole_D2.0mm, F.Cu at (289.7, 110.5)
- added TP9: TestPoint, TestPoint:TestPoint_Plated_Hole_D2.0mm, F.Cu at (294.7, 95.4)
- J1: value Conn_01x06_Pin -> Conn_01x07_Pin; footprint Connector_PinHeader_2.54mm:PinHeader_1x06_P2.54mm_Vertical -> Connector_PinSocket_2.54mm:PinSocket_1x07_P2.54mm_Vertical
- moved J1 28.7 mm to (243.3, 120.0)
- moved R5 0.38 mm to (237.2, 137.8)
Connections:
- J1 pad 1: INB1 -> INB2
- R1 pad 1: Net-(J2-Pin_2) -> Net-(J1-Pin_2)
- R12 pad 1: Net-(J2-Pin_4) -> Net-(J1-Pin_4)
- R4 pad 1: Net-(J1-Pin_4) -> Net-(J6-Pin_4)
- R5 pad 1: Net-(J1-Pin_2) -> Net-(J6-Pin_2)
- R6 pad 1: Net-(J1-Pin_2) -> Net-(J6-Pin_2)
- R8 pad 1: Net-(J2-Pin_2) -> Net-(J1-Pin_2)
- U1 pad 6: Net-(J2-Pin_3) -> Net-(J1-Pin_3)
- U1 pad 7: +3V_1 -> Net-(U1-PWM)
- U2 pad 6: Net-(J1-Pin_3) -> Net-(J6-Pin_3)
- U2 pad 7: +3V_1 -> Net-(U2-PWM)
Routing:
- net Net-(J6-Pin_2): track 0.00 -> 23.6 mm
- net Net-(J2-Pin_2): track 19.9 -> 0.00 mm
- net Net-(J2-Pin_3): track 18.1 -> 0.00 mm
- net Net-(J1-Pin_2): track 19.7 -> 2.21 mm
- net +3V_1: track 75.3 -> 63.5 mm, vias 4 -> 2
- net Net-(J6-Pin_3): track 0.00 -> 8.77 mm
- net INB2: track 40.2 -> 32.3 mm
- net Net-(J1-Pin_7): track 0.00 -> 7.18 mm
- net Net-(J6-Pin_4): track 0.00 -> 6.76 mm
- net Net-(J6-Pin_7): track 0.00 -> 6.74 mm
- net Net-(J2-Pin_4): track 5.74 -> 0.00 mm
- net GND1: track 8.63 -> 14.1 mm
- net Net-(U2-PWM): track 0.00 -> 5.26 mm, vias 0 -> 1
- net INB1: track 39.7 -> 44.9 mm
- net Net-(U1-PWM): track 0.00 -> 4.98 mm, vias 0 -> 1
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Other:
- board text added: "24V 20A"
- board text removed: "24V 30A"

Commit message: version v2.0.0
Parts:
- removed TP1, TP2, TP7: TestPoint, TestPoint:TestPoint_Pad_D1.5mm
- removed TP10, TP11, TP8, TP9: TestPoint, TestPoint:TestPoint_Plated_Hole_D2.0mm
- added INA: TestPoint, TestPoint:TestPoint_Pad_D1.5mm, F.Cu at (237.2, 151.9)
- added INA: TestPoint, TestPoint:TestPoint_Pad_D1.5mm, F.Cu at (234.1, 118.0)
- added INB: TestPoint, TestPoint:TestPoint_Pad_D1.5mm, F.Cu at (240.3, 151.2)
- added OUTA: TestPoint, TP:TestPoint_THTPad_D3.0mm_Drill1.5mm, F.Cu at (198.6, 113.1)
- added OUTA: TestPoint, TP:TestPoint_THTPad_D3.0mm_Drill1.5mm, F.Cu at (222.4, 148.5)
- added OUTB: TestPoint, TP:TestPoint_THTPad_D3.0mm_Drill1.5mm, F.Cu at (193.5, 113.1)
- added OUTB: TestPoint, TP:TestPoint_THTPad_D3.0mm_Drill1.5mm, F.Cu at (207.3, 150.4)
- J10, J5: footprint XT30UPB-M:AMASS_XT30UPB-M -> xt30:xt30
- R14, R15: value 1k -> 100
- TP12, TP3: footprint TestPoint:TestPoint_Plated_Hole_D2.0mm -> TP:TestPoint_THTPad_D3.0mm_Drill1.5mm
- moved G*** 28.0 mm to (236.5, 152.8)
- moved INB 6.47 mm to (240.1, 120.4)
- moved R16 4.70 mm to (237.3, 105.8)
- moved R15 4.68 mm to (240.2, 104.8)
- moved R14 4.32 mm to (240.2, 136.0)
- moved R13 4.30 mm to (237.3, 137.0)
- moved J5 0.73 mm to (196.1, 118.5)
- moved TP12 0.08 mm to (239.3, 88.1)
- moved TP3 0.08 mm to (245.9, 88.1)
- renumbered TP4 to GND, TP6 to GND, TP5 to INB
Routing:
- net Net-(J1-Pin_2): track 2.21 -> 21.8 mm
- net Net-(J3-Pin_2): track 24.2 -> 37.2 mm, vias 5 -> 4
- net INB2: track 32.3 -> 41.7 mm
- net Net-(J6-Pin_3): track 8.77 -> 17.9 mm
- net Net-(J4-Pin_2): track 25.2 -> 34.0 mm, vias 12 -> 15
- net Net-(J5-PadP): track 10.6 -> 18.0 mm, vias 33 -> 26
- net INA2: track 21.3 -> 16.2 mm
- net Net-(J1-Pin_7): track 7.18 -> 2.18 mm
- net Net-(U1-PWM): track 4.98 -> 9.91 mm
- net Net-(J6-Pin_7): track 6.74 -> 2.15 mm
- net Net-(U2-PWM): track 5.26 -> 9.69 mm
- net Net-(J1-Pin_3): track 14.4 -> 18.7 mm
- net +3V_1: track 63.5 -> 59.4 mm
- net GND1: track 14.1 -> 18.2 mm
- net Net-(J10-PadP): track 16.2 -> 12.7 mm, vias 27 -> 20
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Other:
- board text added: "1"
- board text added: "2"
- board text added: "24/Mar 2026 Iter. 2.0.0"
- board text added: "24V 10A"
- board text added: "< INA/B"
- board text added: "DO NOT PROBE ACROSS INA & INB!"
- board text added: "EN > pulled high (enabled) CS_DIS > floating (CS enabled) PWM > pulled high (DC)"
- board text added: "Lin Lab Wei Yue Yucheng Yang PCB by Kevin Ying ⁨Nikita Lukhanin⁩ Divij Muthu Tofic Esses"
- board text added: "OUT 1"
- board text added: "OUT 2"
- board text removed: "4/Mar 2026 Iter. 1.1.0"
- board text removed: "<<< 15A"
- board text removed: "<<<<<"
- board text removed: "EN > pulled high (enabled) CS_DIS > floating (CS enabled)"
- board text removed: "Lin Lab PCB by Kevin Ying Wei Yue Yucheng Yang"

Commit message: 2.0.1
Parts:
- moved PGND 14.0 mm to (257.7, 95.6)
- moved G*** 0.08 mm to (235.9, 96.9)
- renumbered TP3 to PGND, TP12 to VM
Routing:
- net VM1: track 57.2 -> 55.0 mm
- net PGND1: vias 209 -> 208
- net Net-(Q1-D): vias 60 -> 61
- net Net-(J3-Pin_1): vias 27 -> 25
Other:
- board text added: "24/Mar 2026 Iter. 2.0.1"
- board text added: "< IN(B)"
- board text removed: "24/Mar 2026 Iter. 2.0.0"
- board text removed: "< INA/B"
