File: PCB/PWM_amp/PWM_amp.kicad_sch (KiCad schematic)
At the start: 38 parts, among them J1 Conn_01x06_Pin, J10 XT30UPB-M, J2 Conn_01x06_Pin, J3 Conn_01x02_Pin, J4 Conn_01x02_Pin, J49 XT60PW-M, J5 XT30UPB-M, U1 VNH5019A-E, U2 VNH5019A-E, U3 NC7SVU04P5X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

Commit message: code testing for V2
Parts:
- removed C10, C9: 0.1uF, Capacitor_SMD:C_0805_2012Metric_Pad1.18x1.45mm_HandSolder, symbol Device:C
- added Q1, Q2: FDD8447L, Package_TO_SOT_SMD:TO-252-2, symbol Simulation_SPICE:NMOS
Connections:
- net VM1: now also Q1.3 (S), Q2.3 (S)
- net at C3.1, C8.1, U1.13 (VCC)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: now also Q2.2 (D)
- net at C5.1, C7.1, U2.13 (VCC)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: now also Q1.2 (D)
- net at U2.11 (CP): now also Q1.1 (G)
- net at U1.11 (CP): now also Q2.1 (G)
Other:
- moved on the sheet: C3, C5, C7, C8

Commit message: added circuits
Other:
- note added: "This is the PWM driver for the flying robot coil arrays. We want to drive up to 2A per coil continuously at 12V. So for a four-coil unit, you need 8A per driver!"
- note removed: "This is the PWM driver for the flyiing robot coil arrays. We want to drive up to 2A per coil continuously at 12V. So for a four-coil unit, you need 8A per driver at 12V!"
- company: Kevin Ying - Lin Lab -> Micro Flying Robots - Liwei Lin Lab
- moved on the sheet: C1, C2, C3, C4, C5, C6, C7, C8, D1, H1, H2, H3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
