File: PCB/PWM_amp/PWM_amp.kicad_sch (KiCad schematic)
At the start: 54 parts, among them J1 Conn_01x06_Pin, J10 XT30UPB-M, J2 Conn_01x06_Pin, J3 Conn_01x02_Pin, J4 Conn_01x02_Pin, J49 XT60PW-M, J5 XT30UPB-M, Q1 FDD8447L, Q2 FDD8447L, U1 VNH5019A-E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

Commit message: 3d models and PCB
Parts:
- removed H4, H6, H7, H9: MountingHole, MountingHole:MountingHole_3.2mm_M3, symbol Mechanical:MountingHole
- removed TP1: GND1, TestPoint:TestPoint_Loop_D1.80mm_Drill1.0mm_Beaded, symbol Connector:TestPoint
- removed TP10: INA2, TestPoint:TestPoint_Loop_D1.80mm_Drill1.0mm_Beaded, symbol Connector:TestPoint
- removed TP11: INB1, TestPoint:TestPoint_Loop_D1.80mm_Drill1.0mm_Beaded, symbol Connector:TestPoint
- removed TP12: INB2, TestPoint:TestPoint_Loop_D1.80mm_Drill1.0mm_Beaded, symbol Connector:TestPoint
- removed TP13, TP5: EN, TestPoint:TestPoint_Loop_D1.80mm_Drill1.0mm_Beaded, symbol Connector:TestPoint
- removed TP14, TP2: CS, TestPoint:TestPoint_Loop_D1.80mm_Drill1.0mm_Beaded, symbol Connector:TestPoint
- removed TP15, TP4: OUTA, TestPoint:TestPoint_Loop_D1.80mm_Drill1.0mm_Beaded, symbol Connector:TestPoint
- removed TP16, TP3: OUTB, TestPoint:TestPoint_Loop_D1.80mm_Drill1.0mm_Beaded, symbol Connector:TestPoint
- removed TP6: 3V3, TestPoint:TestPoint_Loop_D1.80mm_Drill1.0mm_Beaded, symbol Connector:TestPoint
- removed TP7, TP8: VM1, TestPoint:TestPoint_Loop_D1.80mm_Drill1.0mm_Beaded, symbol Connector:TestPoint
- removed TP9: INA1, TestPoint:TestPoint_Loop_D1.80mm_Drill1.0mm_Beaded, symbol Connector:TestPoint
- added C4, C6: 1uF, Capacitor_SMD:C_0805_2012Metric_Pad1.18x1.45mm_HandSolder, symbol Device:C
- added C7, C8: 0.1uF, Capacitor_SMD:C_0805_2012Metric_Pad1.18x1.45mm_HandSolder, symbol Device:C
Connections:
- net +3V_1: now also J2.5 (Pin_5); no longer J2.4 (Pin_4), R12.1, R4.1
- net GND1: now also J2.6 (Pin_6), R7.1, R9.1; no longer J2.5 (Pin_5)
- net INB2: now also J2.1 (Pin_1); no longer J2.6 (Pin_6)
- net PGND1: now also C4.2, C6.2, C7.2, C8.2
- net VM1: now also C4.1, C6.1
- net at C3.1, Q2.2 (D), U1.13 (VCC)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: now also C8.1
- net at C5.1, Q1.2 (D), U2.13 (VCC)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: now also C7.1
- net at J2.2 (Pin_2): now also R1.1, R8.1; no longer R9.1
- net at R12.2, R9.2: now also U1.8 (CS); no longer U1.6 (CS_DIS)
- net at J1.4 (Pin_4): now also R4.1; no longer U2.8 (CS)
- net at J2.3 (Pin_3): now also U1.6 (CS_DIS); no longer U1.8 (CS)
- net at R4.2, R7.2: now also U2.8 (CS); no longer U2.6 (CS_DIS)
- net at J1.3 (Pin_3): now also U2.6 (CS_DIS); no longer R7.1
- new net: J2.4 (Pin_4), R12.1
Other:
- moved on the sheet: J2, J3, J4, R4, R7, R9

Commit message: DONE DRAFT
Parts:
- removed J1, J2: Conn_01x06_Pin, Connector_PinHeader_2.54mm:PinHeader_1x06_P2.54mm_Vertical, symbol Connector:Conn_01x06_Pin
- added J1, J6: Conn_01x07_Pin, Connector_PinSocket_2.54mm:PinSocket_1x07_P2.54mm_Vertical, symbol Connector:Conn_01x07_Pin
- added R13, R16: 4.7k, Resistor_SMD:R_0805_2012Metric_Pad1.20x1.40mm_HandSolder, symbol Device:R
- added R14, R15: 1k, Resistor_SMD:R_0805_2012Metric_Pad1.20x1.40mm_HandSolder, symbol Device:R
- added TP1, TP2, TP4, TP5, TP6, TP7: TestPoint, TestPoint:TestPoint_Pad_D1.5mm, symbol Connector:TestPoint
- added TP10, TP11, TP12, TP3, TP8, TP9: TestPoint, TestPoint:TestPoint_Plated_Hole_D2.0mm, symbol Connector:TestPoint
Connections:
- net +3V_1: now also J1.5 (Pin_5), J6.5 (Pin_5), R13.2, R16.2; no longer U1.7 (PWM), U2.7 (PWM)
- net GND1: now also J1.6 (Pin_6), J6.6 (Pin_6), TP4.1, TP6.1
- net INA1: now also TP2.1
- net INA2: now also TP7.1
- net INB1: now also J6.1 (Pin_1), TP1.1
- net INB2: now also J1.1 (Pin_1), TP5.1
- net PGND1: now also TP3.1
- net VM1: now also TP12.1
- net at R5.1, R6.1: now also J6.2 (Pin_2)
- net at J3.2 (Pin_2), J5.N: now also TP10.1
- net at R12.1: now also J1.4 (Pin_4)
- net at J5.P, U1.1 (OUTA), U1.25 (OUTA)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: now also TP11.1
- net at R4.1: now also J6.4 (Pin_4)
- net at R1.1, R8.1: now also J1.2 (Pin_2)
- net at U2.6 (CS_DIS): now also J6.3 (Pin_3)
- net at U1.6 (CS_DIS): now also J1.3 (Pin_3)
- new net: J1.7 (Pin_7), R15.1
- new net: R15.2, R16.1, TP9.1, U1.7 (PWM)
- new net: J6.7 (Pin_7), R14.1
- new net: R13.1, R14.2, TP8.1, U2.7 (PWM)
Other:
- note added: "PWM pin pulled high (DC) CS_DIS pulled high to disable. Setting pin3 to low will enable it."
- note removed: "CS_DIS pulled high to disable. Setting pin3 to low will enable it."
- moved on the sheet: R10, R11, R2, R3, U3, U4

Commit message: version v2.0.0
Parts:
- removed TP8, TP9: TestPoint, TestPoint:TestPoint_Plated_Hole_D2.0mm, symbol Connector:TestPoint
- added OUTA1, OUTB1: TestPoint, TP:TestPoint_THTPad_D3.0mm_Drill1.5mm, symbol Connector:TestPoint
- J10, J5: footprint XT30UPB-M:AMASS_XT30UPB-M -> xt30:xt30
- OUTA2: renamed from TP11; footprint TestPoint:TestPoint_Plated_Hole_D2.0mm -> TP:TestPoint_THTPad_D3.0mm_Drill1.5mm
- OUTB2: renamed from TP10; footprint TestPoint:TestPoint_Plated_Hole_D2.0mm -> TP:TestPoint_THTPad_D3.0mm_Drill1.5mm
- R14, R15: value 1k -> 100
- TP12, TP3: footprint TestPoint:TestPoint_Plated_Hole_D2.0mm -> TP:TestPoint_THTPad_D3.0mm_Drill1.5mm
Connections:
- net at J10.N, J4.2 (Pin_2): now also OUTB1.1
- net at J10.P, U2.1 (OUTA), U2.25 (OUTA)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: now also OUTA1.1

Commit message: cleaned up schematic
Other:
- note added: "Bulk Capacitor"
- note added: "This is the pulse-width modulation (PWM) driver to actuate the magnetic coil arrays for the aerial robotics platform. To achieve the required magnetic field strength, the system was specified to drive a continuous current of 2 A per coil at a nominal voltage of 12 V. Consequently, to support the four-coil cluster architecture, each driver unit was engineered to sustain an aggregate continuous cur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"
- note removed: "Bulk Capacitor (idk why)"
- note removed: "This is the PWM driver for the flyiing robot coil arrays. We want to drive up to 2A per coil continuously at 12V. So for a four-coil unit, you need 8A per driver at 12V!"
- company: Kevin Ying - Lin Lab -> UC Berkeley, Liwei Lin Lab
- title: PWM Driver -> Two-Channel Magnetic Coil PWM Driver
- moved on the sheet: C1, C2, C3, C4, C5, C6, C7, C8, D1, H1, H2, H3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
